File: KeyboardPCB/KeyboardPCB.kicad_pcb (KiCad board)
At the start: 2 copper layers, 420 x 297 mm, 73 parts, among them U1 Arduino_Pro_Micro

Commit message: Adding push button with caps 3D model
Parts:
- S1, S10, S11, S12, S13, S14, S15, S16, S17, S18, S19, S2, S20, S21, S22, S23, S24, S25, S26, S27, S28, S29, S3, S30, S31, S32, S33, S34, S35, S36, S4, S5, S6, S7, S8, S9: footprint Button_Switch_THT:SW_PUSH-12mm -> SW_PUSH-WITHCAP-12mm:SW_PUSH-WITHCAP-12mm

Commit message: Arranging button positions
Parts:
- D10, D11, D12, D13, D14, D15, D16, D17, D18, D19, D2, D20, D21, D22, D23, D24, D25, D26, D27, D28, D29, D3, D30, D4, D5, D6, D7, D8, D9: moved to B.Cu
- moved D31 289.2 mm to (100.0, 330.0)
- moved S31 288.5 mm to (80.0, 330.0)
- moved D32 257.7 mm to (140.0, 330.0)
- moved S12 256.3 mm to (450.0, 100.0)
- moved S32 250.1 mm to (120.0, 330.0)
- moved S18 230.1 mm to (450.0, 130.0)
- moved D33 228.8 mm to (180.0, 330.0)
- moved S6 228.1 mm to (450.0, 70.0)
- moved S33 213.4 mm to (160.0, 330.0)
- moved S24 206.2 mm to (450.0, 160.0)
- moved D34 203.9 mm to (220.0, 330.0)
- moved D25 199.4 mm to (140.0, 207.6), turned to 90 degrees
- moved D6 189.2 mm to (480.0, 87.6), turned to 90 degrees
- moved D12 187.1 mm to (480.0, 117.6), turned to 90 degrees
- moved S11 186.3 mm to (380.0, 100.0)
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Connections:
- S15 pad 1: unconnected-(S15-Pad1) -> Column 2
- S21 pad 1: unconnected-(S21-Pad1) -> Column 2
- S27 pad 1: unconnected-(S27-Pad1) -> Column 2
- S33 pad 1: unconnected-(S33-Pad1) -> Column 2
- S9 pad 1: unconnected-(S9-Pad1) -> Column 2
