File: KeyboardPCB/KeyboardPCB.kicad_sch (KiCad schematic)
At the start: 73 parts, among them U1 Arduino_Pro_Micro

Commit message: Adding push button with caps 3D model
Parts:
- S1, S10, S11, S12, S13, S14, S15, S16, S17, S18, S19, S2, S20, S21, S22, S23, S24, S25, S26, S27, S28, S29, S3, S30, S31, S32, S33, S34, S35, S36, S4, S5, S6, S7, S8, S9: footprint Button_Switch_THT:SW_PUSH-12mm -> SW_PUSH-WITHCAP-12mm:SW_PUSH-WITHCAP-12mm
Connections:
- net Row 2 is gone; now on net Column 4: D13.1 (K), D14.1 (K), D15.1 (K), D16.1 (K), D17.1 (K), D18.1 (K), U1.7 (4/PD4)
Changed lines of the file:
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@@
 		)
 	)
+	(label "Row 2"
+		(at 176.53 83.82 0)
+		(effects
+			(font
+				(size 1.27 1.27)
+			)
+			(justify left bottom)
+		)
+	)
 	(global_label "Column 5"
 		(shape input)
@@
 			)
 		)
-		(property "Footprint" "Button_Switch_THT:SW_PUSH-12mm"
+		(property "Footprint" "SW_PUSH-WITHCAP-12mm:SW_PUSH-WITHCAP-12mm"
 			(at 102.87 111.76 0)
 			(effects
@@
 			)
 		)
-		(property "Footprint" "Button_Switch_THT:SW_PUSH-12mm"
+		(property "Footprint" "SW_PUSH-WITHCAP-12mm:SW_PUSH-WITHCAP-12mm"
 			(at 179.07 73.66 0)
 			(effects
@@
 			)
 		)
-		(property "Footprint" "Button_Switch_THT:SW_PUSH-12mm"
+		(property "Footprint" "SW_PUSH-WITHCAP-12mm:SW_PUSH-WITHCAP-12mm"
 			(at 26.67 35.56 0)
 			(effects
@@
 			)
 		)
-		(property "Footprint" "Button_Switch_THT:SW_PUSH-12mm"
+		(property "Footprint" "SW_PUSH-WITHCAP-12mm:SW_PUSH-WITHCAP-12mm"
 			(at 217.17 54.61 0)
 			(effects
@@
 			)
 		)
-		(property "Footprint" "Button_Switch_THT:SW_PUSH-12mm"
+		(property "Footprint" "SW_PUSH-WITHCAP-12mm:SW_PUSH-WITHCAP-12mm"
 			(at 217.17 73.66 0)
 			(effects
@@
 			)
 		)
-		(property "Footprint" "Button_Switch_THT:SW_PUSH-12mm"
+		(property "Footprint" "SW_PUSH-WITHCAP-12mm:SW_PUSH-WITHCAP-12mm"
 			(at 26.67 130.81 0)
 			(effects
@@
 			)
 		)
-		(property "Footprint" "Button_Switch_THT:SW_PUSH-12mm"
+		(property "Footprint" "SW_PUSH-WITHCAP-12mm:SW_PUSH-WITHCAP-12mm"
 			(at 26.67 54.61 0)
 			(effects
@@
 			)
 		)
-		(property "Footprint" "Button_Switch_THT:SW_PUSH-12mm"
+		(property "Footprint" "SW_PUSH-WITHCAP-12mm:SW_PUSH-WITHCAP-12mm"
 			(at 217.17 111.76 0)
 			(effects
@@
 			)
 		)
-		(property "Footprint" "Button_Switch_THT:SW_PUSH-12mm"
+		(property "Footprint" "SW_PUSH-WITHCAP-12mm:SW_PUSH-WITHCAP-12mm"
 			(at 64.77 35.56 0)
 			(effects
@@
 			)
 		)
-		(property "Footprint" "Button_Switch_THT:SW_PUSH-12mm"
+		(property "Footprint" "SW_PUSH-WITHCAP-12mm:SW_PUSH-WITHCAP-12mm"
 			(at 102.87 73.66 0)
 			(effects
@@
 			)
 		)
-		(property "Footprint" "Button_Switch_THT:SW_PUSH-12mm"
+		(property "Footprint" "SW_PUSH-WITHCAP-12mm:SW_PUSH-WITHCAP-12mm"
 			(at 140.97 73.66 0)
 			(effects
@@
 			)
 		)
-		(property "Footprint" "Button_Switch_THT:SW_PUSH-12mm"
+		(property "Footprint" "SW_PUSH-WITHCAP-12mm:SW_PUSH-WITHCAP-12mm"
 			(at 179.07 130.81 0)
 			(effects
@@
 			)
 		)
-		(property "Footprint" "Button_Switch_THT:SW_PUSH-12mm"
+		(property "Footprint" "SW_PUSH-WITHCAP-12mm:SW_PUSH-WITHCAP-12mm"
 			(at 217.17 130.81 0)
 			(effects
@@
 			)
 		)
-		(property "Footprint" "Button_Switch_THT:SW_PUSH-12mm"
+		(property "Footprint" "SW_PUSH-WITHCAP-12mm:SW_PUSH-WITHCAP-12mm"
 			(at 64.77 54.61 0)
 			(effects
@@
 			)
 		)
-		(property "Footprint" "Button_Switch_THT:SW_PUSH-12mm"
+		(property "Footprint" "SW_PUSH-WITHCAP-12mm:SW_PUSH-WITHCAP-12mm"
 			(at 102.87 130.81 0)
 			(effects
@@
 			)
 		)
-		(property "Footprint" "Button_Switch_THT:SW_PUSH-12mm"
+		(property "Footprint" "SW_PUSH-WITHCAP-12mm:SW_PUSH-WITHCAP-12mm"
 			(at 102.87 35.56 0)
 			(effects
@@
 			)
 		)
-		(property "Footprint" "Button_Switch_THT:SW_PUSH-12mm"
+		(property "Footprint" "SW_PUSH-WITHCAP-12mm:SW_PUSH-WITHCAP-12mm"
 			(at 102.87 92.71 0)
 			(effects
@@
 			)
 		)
-		(property "Footprint" "Button_Switch_THT:SW_PUSH-12mm"
+		(property "Footprint" "SW_PUSH-WITHCAP-12mm:SW_PUSH-WITHCAP-12mm"
 			(at 179.07 54.61 0)
 			(effects
@@
 			)
 		)
-		(property "Footprint" "Button_Switch_THT:SW_PUSH-12mm"
+		(property "Footprint" "SW_PUSH-WITHCAP-12mm:SW_PUSH-WITHCAP-12mm"
 			(at 26.67 111.76 0)
 			(effects
@@
 			)
 		)
-		(property "Footprint" "Button_Switch_THT:SW_PUSH-12mm"
+		(property "Footprint" "SW_PUSH-WITHCAP-12mm:SW_PUSH-WITHCAP-12mm"
 			(at 140.97 35.56 0)
 			(effects
@@
 			)
 		)
-		(property "Footprint" "Button_Switch_THT:SW_PUSH-12mm"
+		(property "Footprint" "SW_PUSH-WITHCAP-12mm:SW_PUSH-WITHCAP-12mm"
 			(at 26.67 73.66 0)
 			(effects
@@
 			)
 		)
-		(property "Footprint" "Button_Switch_THT:SW_PUSH-12mm"
+		(property "Footprint" "SW_PUSH-WITHCAP-12mm:SW_PUSH-WITHCAP-12mm"
 			(at 217.17 92.71 0)
 			(effects
@@
 			)
 		)
-		(property "Footprint" "Button_Switch_THT:SW_PUSH-12mm"
+		(property "Footprint" "SW_PUSH-WITHCAP-12mm:SW_PUSH-WITHCAP-12mm"
 			(at 140.97 54.61 0)
 			(effects
@@
 			)
 		)
-		(property "Footprint" "Button_Switch_THT:SW_PUSH-12mm"
+		(property "Footprint" "SW_PUSH-WITHCAP-12mm:SW_PUSH-WITHCAP-12mm"
 			(at 179.07 111.76 0)
 			(effects
@@
 			)
 		)
-		(property "Footprint" "Button_Switch_THT:SW_PUSH-12mm"
+		(property "Footprint" "SW_PUSH-WITHCAP-12mm:SW_PUSH-WITHCAP-12mm"
 			(at 26.67 92.71 0)
 			(effects
@@
 			)
 		)
-		(property "Footprint" "Button_Switch_THT:SW_PUSH-12mm"
+		(property "Footprint" "SW_PUSH-WITHCAP-12mm:SW_PUSH-WITHCAP-12mm"
 			(at 64.77 111.76 0)
 			(effects
@@
 			)
 		)
-		(property "Footprint" "Button_Switch_THT:SW_PUSH-12mm"
+		(property "Footprint" "SW_PUSH-WITHCAP-12mm:SW_PUSH-WITHCAP-12mm"
 			(at 64.77 130.81 0)
 			(effects
@@
 			)
 		)
-		(property "Footprint" "Button_Switch_THT:SW_PUSH-12mm"
+		(property "Footprint" "SW_PUSH-WITHCAP-12mm:SW_PUSH-WITHCAP-12mm"
 			(at 64.77 92.71 0)
 			(effects
@@
 			)
 		)
-		(property "Footprint" "Button_Switch_THT:SW_PUSH-12mm"
+		(property "Footprint" "SW_PUSH-WITHCAP-12mm:SW_PUSH-WITHCAP-12mm"
 			(at 140.97 130.81 0)
 			(effects
@@
 			)
 		)
-		(property "Footprint" "Button_Switch_THT:SW_PUSH-12mm"
+		(property "Footprint" "SW_PUSH-WITHCAP-12mm:SW_PUSH-WITHCAP-12mm"
 			(at 140.97 111.76 0)
 			(effects
@@
 			)
 		)
-		(property "Footprint" "Button_Switch_THT:SW_PUSH-12mm"
+		(property "Footprint" "SW_PUSH-WITHCAP-12mm:SW_PUSH-WITHCAP-12mm"
 			(at 217.17 35.56 0)
 			(effects
@@
 			)
 		)
-		(property "Footprint" "Button_Switch_THT:SW_PUSH-12mm"
+		(property "Footprint" "SW_PUSH-WITHCAP-12mm:SW_PUSH-WITHCAP-12mm"
 			(at 102.87 54.61 0)
 			(effects
@@
 			)
 		)
-		(property "Footprint" "Button_Switch_THT:SW_PUSH-12mm"
+		(property "Footprint" "SW_PUSH-WITHCAP-12mm:SW_PUSH-WITHCAP-12mm"
 			(at 64.77 73.66 0)
 			(effects
@@
 			)
 		)
-		(property "Footprint" "Button_Switch_THT:SW_PUSH-12mm"
+		(property "Footprint" "SW_PUSH-WITHCAP-12mm:SW_PUSH-WITHCAP-12mm"
 			(at 140.97 92.71 0)
 			(effects
@@
 			)
 		)
-		(property "Footprint" "Button_Switch_THT:SW_PUSH-12mm"
+		(property "Footprint" "SW_PUSH-WITHCAP-12mm:SW_PUSH-WITHCAP-12mm"
 			(at 179.07 92.71 0)
 			(effects
@@
 			)
 		)
-		(property "Footprint" "Button_Switch_THT:SW_PUSH-12mm"
+		(property "Footprint" "SW_PUSH-WITHCAP-12mm:SW_PUSH-WITHCAP-12mm"
 			(at 179.07 35.56 0)
 			(effects

Commit message: Arranging button positions
Connections:
- net Column 2: now also S15.1, S21.1, S27.1, S33.1, S9.1
Changed lines of the file:
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@@
+	)
+	(junction
+		(at 100.33 52.07)
+		(diameter 0)
+		(color 0 0 0 0)
 	)
 	(junction
@@
 	)
 	(junction
+		(at 100.33 90.17)
+		(diameter 0)
+		(color 0 0 0 0)
+	)
+	(junction
 		(at 105.41 64.77)
 		(diameter 0)
@@
 	)
 	(junction
+		(at 100.33 109.22)
+		(diameter 0)
+		(color 0 0 0 0)
+	)
+	(junction
 		(at 105.41 45.72)
 		(diameter 0)
@@
 	)
 	(junction
+		(at 100.33 33.02)
+		(diameter 0)
+		(color 0 0 0 0)
+	)
+	(junction
 		(at 24.13 71.12)
 		(diameter 0)
@@
 	)
 	(junction
+		(at 100.33 71.12)
+		(diameter 0)
+		(color 0 0 0 0)
+	)
+	(junction
 		(at 219.71 64.77)
 		(diameter 0)
@@
 	(wire
 		(pts
+			(xy 100.33 90.17) (xy 100.33 109.22)
+		)
+		(stroke
+			(width 0)
+			(type default)
+		)
+	)
+	(wire
+		(pts
 			(xy 176.53 90.17) (xy 176.53 109.22)
 		)
@@
 	(wire
 		(pts
+			(xy 100.33 52.07) (xy 100.33 71.12)
+		)
+		(stroke
+			(width 0)
+			(type default)
+		)
+	)
+	(wire
+		(pts
 			(xy 219.71 45.72) (xy 228.6 45.72)
 		)
@@
 	(wire
 		(pts
+			(xy 100.33 33.02) (xy 100.33 52.07)
+		)
+		(stroke
+			(width 0)
+			(type default)
+		)
+	)
+	(wire
+		(pts
 			(xy 62.23 52.07) (xy 62.23 71.12)
 		)
@@
 	(wire
 		(pts
+			(xy 100.33 71.12) (xy 100.33 90.17)
+		)
+		(stroke
+			(width 0)
+			(type default)
+		)
+	)
+	(wire
+		(pts
 			(xy 24.13 109.22) (xy 24.13 128.27)
 		)
@@
 		)
 		(stroke
+			(width 0)
+			(type default)
+		)
+	)
+	(wire
+		(pts
+			(xy 100.33 109.22) (xy 100.33 128.27)
+		)
+		(stroke
